Commit message: Added an rviz configuration.

File: urdf/slidebot.urdf (robot description, URDF)
Before this commit: robot slidebot, 1 links, 0 joints
Links:
- removed link base
- added link base_link; visual box size=3 2 1

Commit message: Created a more complete robot.

File: urdf/slidebot.urdf (robot description, URDF)
Before this commit: robot slidebot, 1 links, 0 joints
Links:
- removed link base_link
- added link arm; visual cylinder length=1.0 radius=0.1
- added link base; visual sphere radius=0.1
- added link body; visual box size=3 2 1
Joints:
- added joint linear: type prismatic, parent base, child body, limit lower=-10 upper=10 effort=100 velocity=100
- added joint rotational: type continuous, parent body, child arm, origin xyz=1.5 0 0.5 rpy=0 0 0

Commit message: Updated for ROS2

File: urdf/slidebot.urdf (robot description, URDF)
Before this commit: robot slidebot, 3 links, 2 joints
Links:
- removed link base
- added link base_link; visual sphere radius=0.1
Joints:
- joint linear: parent base -> base_link
