Commit message: Fixed typo

File: urdf/chain_link.urdf.xacro (robot description, xacro)
@@ -11,8 +11,8 @@
       </geometry>
     </collision>
-    <intertial>
+    <inertial>
       <mass value="1"/>
-      <intertia ixx="${radius**2/2.0}" iyy="${(length**2 + 3.0*radius**2)/12.0}" izz="${(length**2 + 3.0*radius**2)/12.0}" ixy="0.0" ixz="0.0" iyz="0.0" />
-    </intertial>
+      <inertia ixx="${radius**2/2.0}" iyy="${(length**2 + 3.0*radius**2)/12.0}" izz="${(length**2 + 3.0*radius**2)/12.0}" ixy="0.0" ixz="0.0" iyz="0.0" />
+    </inertial>
   </xacro:macro>
 </robot>
